File: RTN-Badge-NL-2026.kicad_sch (KiCad schematic)
At the start: 20 parts, among them J1 USB_A_Edge_Connector, J2 DEBUG, J3 GPIO, SW1 BOOT, SW2 RST, SW3 USER1, SW4 USER2, U1 CH32V203F6P6, U2 XC6206PxxxMR, Y1 8MHz

Commit message: Add grounded mounting holes
Parts:
- added H1, H2, H3: MountingHole_Pad, MountingHole:MountingHole_2.2mm_M2_Pad_Via, symbol Mechanical:MountingHole_Pad
Connections:
- net GND: now also H1.1, H2.1, H3.1
